Commit message: add files for lecture 2024

File: doosan-robot/dsr_description/urdf/m0609_robotiq_2f_85.urdf (robot description, URDF)
Before this commit: robot m0609_robotiq_2f_85, 18 links, 17 joints
Links:
- added link robotiq_virtual_base_link
- added link robotiq_virtual_link
Joints:
- added joint robotiq_virtual_base_joint: type fixed, parent link6, child robotiq_virtual_base_link, origin xyz=0 0 0.115 rpy=0 0 0
- added joint robotiq_virtual_joint: type fixed, parent robotiq_virtual_base_link, child robotiq_virtual_link, origin xyz=0 0 0 rpy=3.141592653589793 0 0
